File: Octoprober.brd (EAGLE design)
At the start: 130.8 x 95 mm, 147 parts, among them J1 10118193-0001LF, J2 26-60-4020, SW1 EVQ-Q2203W, SW2 EVQ-Q2203W, SW3 EVQ-Q2203W, SW4 EVQ-Q2203W, SW5 EVQ-Q2203W, U1 P8X32A-M44, U10 MAX31855KASA+, U11 MAX31855KASA+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

Commit message: REV1 finished routing. Need to increase font size.
Parts:
- added R34: 120, PP_Passives:0402
- J2: value 26-60-4020 -> (none); device PP_Connectors:MOLEX_KK_2 -> PP_Connectors:HEADER_01X04_PTH
- moved C11 2.03 mm to (112.3, 91.9)
- moved C13 2.03 mm to (110.4, 91.9)
- moved D1 2.03 mm to (102.1, 91.9)
- moved D2 2.03 mm to (105.9, 91.9)
- moved R12 2.03 mm to (107.8, 91.9)
- moved R13 2.03 mm to (104.0, 91.9)
- moved J2 1.25 mm to (100.8, 7.87), turned to 180 degrees
Connections:
- net EXT renamed EXT0
- removed net P26: U1.33
- new net EXT1: OP1.3, U1.33
- new net EXT_CON_2: J2.3, OP1.6
- new net EXT_CON_3: J2.4, OP1.5
- new net N$24: OP1.4, R34.2
- net EXT_CON_0: now also J2.1; no longer J2.P$2
- net EXT_CON_1: now also J2.2; no longer J2.P$1
- net GND: now also R34.1
Routing:
- net EXT1: track 0.00 -> 31.1 mm
- net EXT_CON_3: track 0.00 -> 12.3 mm
- net EXT_CON_2: track 0.00 -> 11.8 mm
- net !PWREN: track 196.2 -> 200.3 mm
- net FT230_RST: track 49.4 -> 53.5 mm
- net !SLEEP: track 201.7 -> 205.8 mm
- net N$24: track 0.00 -> 2.73 mm
- net TXRX_LED: track 6.14 -> 8.17 mm
- net 3V3OUT: track 19.4 -> 21.4 mm
- net EXT_CON_0: track 9.06 -> 10.7 mm
- net EXT_CON_1: track 9.82 -> 11.2 mm
- net N$4: track 110.6 -> 109.3 mm
- net USB_V1: track 227.7 -> 228.2 mm
- net GND: track 400.2 -> 400.7 mm, vias 49 -> 50
Other:
- board text added: "+"
- board text added: "-"
