File: Hardware/Octoprober.brd (EAGLE design)
At the start: 183 parts, among them J4 ER-CON31HT-1, SW1 EVQ-Q2203W, SW2 EVQ-Q2203W, SW3 EVQ-Q2203W, SW4 EVQ-Q2203W, SW5 EVQ-Q2203W, T1 PCC-SMP-V, T2 PCC-SMP-V, T3 PCC-SMP-V, T4 PCC-SMP-V, T5 PCC-SMP-V, T6 PCC-SMP-V, T7 PCC-SMP-V, T8 PCC-SMP-V, U1 P8X32A-Q44, U10 BQ24075RGTT, U11 MAX31856MUD+, U12 MAX31856MUD+, U13 MAX31856MUD+, U14 MAX31856MUD+, U15 MAX31856MUD+, U16 MAX31856MUD+, U17 MAX31856MUD+, U18 MAX31856MUD+, U19 IP4234CZ6,125, U2 CAT24C512WI-GT3, U20 PMV160UP,215, U21 74HCT2G04GV,125, U4 FT230XQ-R, U5 ADP3338AKCZ-3.3-RL, U6 DS1340Z-33+, U7 PMV22EN,215, U8 PMV160UP,215, U9 MCP3021A5T-E/OT, X1 ABLS3-6.000MHZ-D4Y-T, X2 ABS25-32.768KHz-1-T

Commit message: Working on new rev. Need to route.
Parts:
- removed J5: (no value), PP_Connectors:2.54MM_01X02_PIN_HEADER
- added BATT1: 1042, PP_Connectors:KEYSTONE_1042
- J6: value (none) -> ER-CON2.0-2P-SMD
- R10, R11: value 22 -> 27
Connections:
- net GND: now also BATT1.N; no longer J5.1
- net LCD_SCL: now also J4.P$16, R39.1; no longer J4.P$11, J4.P$12, J4.P$13, J4.P$15, R38.1
- net LCD_SDA: now also J4.P$11, J4.P$12, J4.P$13, J4.P$15, R38.1; no longer J4.P$16, R39.1
- net VBATT: now also BATT1.P; no longer J5.2
Changed lines of the file:
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@@
 <attribute name="NAME" x="111.287" y="93.5035" size="0.8128" layer="25" font="vector" ratio="16"/>
 </element>
-<element name="R10" library="PP_Passives" package="0603" value="22" x="119.253" y="85.566" smashed="yes" rot="R270">
+<element name="R10" library="PP_Passives" package="0603" value="27" x="119.253" y="85.566" smashed="yes" rot="R270">
 <attribute name="NAME" x="118.399" y="83.0895" size="0.8128" layer="25" font="vector" ratio="16"/>
 </element>
-<element name="R11" library="PP_Passives" package="0603" value="22" x="117.348" y="85.566" smashed="yes" rot="R270">
+<element name="R11" library="PP_Passives" package="0603" value="27" x="117.348" y="85.566" smashed="yes" rot="R270">
 <attribute name="NAME" x="114.589" y="86.0105" size="0.8128" layer="25" font="vector" ratio="16"/>
 </element>
@@
 <attribute name="LABEL14" value="DB5" x="-13.716" y="-242.316" size="1.778" layer="27" display="off"/>
 <attribute name="LABEL30" value="V1" x="-13.716" y="-242.316" size="1.778" layer="27" display="off"/>
-<attribute name="LABEL15" value="DB6_SCL" x="-13.716" y="-242.316" size="1.778" layer="27" display="off"/>
+<attribute name="LABEL15" value="DB6_SDA" x="-13.716" y="-242.316" size="1.778" layer="27" display="off"/>
 <attribute name="LABEL31" value="V0" x="-13.716" y="-242.316" size="1.778" layer="27" display="off"/>
-<attribute name="LABEL16" value="DB7_SDA" x="-13.716" y="-242.316" size="1.778" layer="27" display="off"/>
+<attribute name="LABEL16" value="DB7_SCL" x="-13.716" y="-242.316" size="1.778" layer="27" display="off"/>
 <attribute name="LABEL17" value="VDD" x="-13.716" y="-242.316" size="1.778" layer="27" display="off"/>
 <attribute name="LABEL18" value="VDD" x="-13.716" y="-242.316" size="1.778" layer="27" display="off"/>
@@
 <element name="C79" library="PP_Passives" package="0603" value="1uF" x="-23.114" y="-281.178"/>
 <element name="C80" library="PP_Passives" package="0603" value="3.3uF" x="-23.114" y="-284.48"/>
-<element name="J5" library="PP_Connectors" package="2.54MM_01X02_PIN_HEADER" value="" x="-27.94" y="-276.606">
-<attribute name="LABEL02" value="VBATT+" x="-27.94" y="-276.606" size="1.778" layer="27" display="off"/>
-<attribute name="LABEL01" value="VBATT-" x="-27.94" y="-276.606" size="1.778" layer="27" display="off"/>
-</element>
-<element name="J6" library="PP_Connectors" package="ER-CON2.0-2P-SMD" value="" x="-40.132" y="-276.098">
+<element name="J6" library="PP_Connectors" package="ER-CON2.0-2P-SMD" value="ER-CON2.0-2P-SMD" x="-40.132" y="-276.098">
 <attribute name="LABEL02" value="" x="-40.132" y="-276.098" size="1.778" layer="27" display="off"/>
 <attribute name="LABEL01" value="" x="-40.132" y="-276.098" size="1.778" layer="27" display="off"/>
@@
 <element name="U10" library="PP_PowerIC" package="BQ2407X_VQFN-16" value="BQ24075RGTT" x="-57.658" y="-301.752"/>
 <element name="U5" library="PP_PowerIC" package="ADP3338_SOT-223-3" value="ADP3338AKCZ-3.3-RL" x="-64.516" y="-299.974"/>
+<element name="BATT1" library="PP_Connectors" package="KEYSTONE_1042" value="1042" x="26.924" y="-206.756" rot="R90"/>
 </elements>
 <signals>
@@
 <contactref element="J4" pad="P$2"/>
 <contactref element="J4" pad="P$1"/>
-<contactref element="J5" pad="1"/>
 <contactref element="J6" pad="P$2"/>
 <contactref element="U2" pad="4"/>
@@
 <contactref element="U10" pad="15"/>
 <contactref element="U5" pad="1"/>
+<contactref element="BATT1" pad="N"/>
 <wire x1="112.268" y1="92.766" x2="124.333" y2="86.416" width="0" layer="19" extent="1-1"/>
 <wire x1="110.363" y1="92.766" x2="112.268" y2="92.766" width="0" layer="19" extent="1-1"/>
@@
 <wire x1="-20.716" y1="-242.316" x2="-7.874" y2="-160.894" width="0" layer="19" extent="1-1"/>
 <wire x1="-21.216" y1="-242.316" x2="-20.716" y2="-242.316" width="0" layer="19" extent="1-1"/>
-<wire x1="-29.21" y1="-276.606" x2="-21.216" y2="-242.316" width="0" layer="19" extent="1-1"/>
-<wire x1="-39.132" y1="-276.098" x2="-29.21" y2="-276.606" width="0" layer="19" extent="1-1"/>
+<wire x1="-39.132" y1="-276.098" x2="-21.216" y2="-242.316" width="0" layer="19" extent="1-1"/>
 <wire x1="-47.234" y1="-289.433" x2="-39.132" y2="-276.098" width="0" layer="19" extent="1-1"/>
 <wire x1="-52.334" y1="-289.433" x2="-47.234" y2="-289.433" width="0" layer="19" extent="1-1"/>
@@
 <wire x1="-52.334" y1="-303.657" x2="-56.908" y2="-303.227" width="0" layer="19" extent="1-1"/>
 <wire x1="-66.816" y1="-302.514" x2="-57.908" y2="-300.277" width="0" layer="19" extent="1-1"/>
+<wire x1="26.924" y1="-246.0879" x2="-66.816" y2="-302.514" width="0" layer="19" extent="1-1"/>
 </signal>
 <signal name="RES">
@@
 <contactref element="C31" pad="1"/>
 <contactref element="R29" pad="1"/>
-<contactref element="J5" pad="2"/>
 <contactref element="U10" pad="3"/>
 <contactref element="U10" pad="2"/>
+<contactref element="BATT1" pad="P"/>
 <wire x1="-59.133" y1="-301.502" x2="-59.133" y2="-302.002" width="0" layer="19" extent="1-1"/>
-<wire x1="-26.67" y1="-276.606" x2="-59.133" y2="-301.502" width="0" layer="19" extent="1-1"/>
-<wire x1="49.022" y1="16.602" x2="-26.67" y2="-276.606" width="0" layer="19" extent="1-1"/>
-<wire x1="78.74" y1="8.262" x2="49.022" y2="16.602" width="0" layer="19" extent="1-1"/>
+<wire x1="26.924" y1="-167.4241" x2="-59.133" y2="-302.002" width="0" layer="19" extent="1-1"/>
+<wire x1="78.74" y1="8.262" x2="26.924" y2="-167.4241" width="0" layer="19" extent="1-1"/>
+<wire x1="49.022" y1="16.602" x2="78.74" y2="8.262" width="0" layer="19" extent="1-1"/>
 </signal>
 <signal name="TP_T-_0">
@@
 <signal name="LCD_SCL">
 <contactref element="U1" pad="1"/>
-<contactref element="J4" pad="P$15"/>
+<contactref element="J4" pad="P$16"/>
+<contactref element="R39" pad="1"/>
+<wire x1="-13.716" y1="-242.316" x2="-13.574" y2="-151.194" width="0" layer="19" extent="1-1"/>
+<wire x1="-22.948" y1="-261.874" x2="-13.716" y2="-242.316" width="0" layer="19" extent="1-1"/>
+</signal>
+<signal name="LCD_SDA">
+<contactref element="U1" pad="2"/>
+<contactref element="J4" pad="P$11"/>
 <contactref element="R38" pad="1"/>
-<contactref element="J4" pad="P$11"/>
 <contactref element="J4" pad="P$12"/>
 <contactref element="J4" pad="P$13"/>
-<wire x1="-14.216" y1="-242.316" x2="-13.574" y2="-151.194" width="0" layer="19" extent="1-1"/>
-<wire x1="-15.216" y1="-242.316" x2="-14.216" y2="-242.316" width="0" layer="19" extent="1-1"/>
+<contactref element="J4" pad="P$15"/>
+<wire x1="-15.216" y1="-242.316" x2="-13.574" y2="-151.994" width="0" layer="19" extent="1-1"/>
 <wire x1="-15.716" y1="-242.316" x2="-15.216" y2="-242.316" width="0" layer="19" extent="1-1"/>
 <wire x1="-16.216" y1="-242.316" x2="-15.716" y2="-242.316" width="0" layer="19" extent="1-1"/>
+<wire x1="-14.216" y1="-242.316" x2="-15.216" y2="-242.316" width="0" layer="19" extent="1-1"/>
 <wire x1="-22.948" y1="-258.572" x2="-16.216" y2="-242.316" width="0" layer="19" extent="1-1"/>
 </signal>
-<signal name="LCD_SDA">
-<contactref element="U1" pad="2"/>
-<contactref element="J4" pad="P$16"/>
-<contactref element="R39" pad="1"/>
-<wire x1="-13.716" y1="-242.316" x2="-13.574" y2="-151.994" width="0" layer="19" extent="1-1"/>
-<wire x1="-22.948" y1="-261.874" x2="-13.716" y2="-242.316" width="0" layer="19" extent="1-1"/>
-</signal>
 <signal name="LCD_RST">

Commit message: Started routing REV3.
Parts:
- removed C41: 10uF, PP_Passives:1206
- added C81, C82: 47pF, PP_Passives:0603
- added C83: 0.1uF, PP_Passives:0603
- X1: value ABLS3-6.000MHZ-D4Y-T -> ABMM-6.000MHZ-B2-T; device PP_FreqCtrl:HC-49/US_SM -> MF_Frequency_Control:7MMX5MM
- moved U$4 292.4 mm to (255.8, -171.0)
- moved C1 287.2 mm to (229.6, -242.1)
- moved C23 287.2 mm to (199.9, -189.7)
- moved C31 287.2 mm to (162.8, -245.7)
- moved C32 287.2 mm to (174.2, -245.4)
- moved C33 287.2 mm to (172.7, -241.3)
- moved C34 287.2 mm to (181.6, -245.9)
- moved C35 287.2 mm to (184.4, -245.4)
- moved C36 287.2 mm to (191.0, -248.4)
- moved C38 287.2 mm to (201.9, -253.8)
- moved C39 287.2 mm to (196.6, -254.5)
- moved C45 287.2 mm to (153.9, -240.5)
- moved C53 287.2 mm to (212.1, -195.1)
- moved C7 287.2 mm to (148.3, -255.8)
- moved C8 287.2 mm to (145.3, -255.8)
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Connections:
- net 3.3V: now also C83.1; no longer C41.1
- net D+: now also C82.1
- net D-: now also C81.1
- net GND: now also C81.2, C82.2, C83.2, X1.P$2, X1.P$4; no longer C41.2
- net X0: now also X1.P$3; no longer X1.P$1
- net X1: now also X1.P$1; no longer X1.P$2
Routing:
- net GND: track 0.00 -> 176.8 mm, vias 0 -> 53
- net ADC_SCK: track 0.00 -> 116.7 mm, vias 0 -> 8
- net ADC_SDO: track 0.00 -> 104.2 mm, vias 0 -> 8
- net ADC_SDI: track 0.00 -> 98.6 mm, vias 0 -> 8
- net 3.3V: track 0.00 -> 57.2 mm, vias 0 -> 13
- net 3.3V_ANALOG: track 0.00 -> 53.9 mm, vias 0 -> 16
- net USB_V1: track 0.00 -> 29.7 mm, vias 0 -> 2
- net ADC_3_!CS: track 0.00 -> 28.3 mm
- net ADC_2_!CS: track 0.00 -> 28.2 mm
- net ADC_4_!CS: track 0.00 -> 28.2 mm
- net ADC_1_!CS: track 0.00 -> 28.1 mm
- net ADC_0_!CS: track 0.00 -> 28.1 mm
- net ADC_5_!CS: track 0.00 -> 28.0 mm
- net ADC_6_!CS: track 0.00 -> 27.6 mm
- net ADC_7_!CS: track 0.00 -> 27.6 mm
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- added copper zone on layer 15, net 3.3V
- added copper zone on layer 15, net 3.3V_ANALOG
- added copper zone on layer 2, net GND

Commit message: More work to check in.
Parts:
- removed D2: 598-8070-107F, PP_LED:LED_0805
- removed R12: 330, PP_Passives:0603
- removed U$3, U$4, U$5, U$6: (no value), PP_Connectors:MOUNT_HOLE_2.8MM
- moved R38 83.2 mm to (-11.7, -134.2)
- moved R39 83.2 mm to (-9.91, -134.2)
- moved C75 82.9 mm to (-6.60, -133.4)
- moved C76 82.9 mm to (2.79, -135.9)
- moved C77 82.9 mm to (1.27, -135.9)
- moved C78 82.9 mm to (-0.25, -135.9)
- moved C79 82.9 mm to (-1.78, -135.9)
- moved C80 82.9 mm to (-3.30, -135.9)
- moved J6 82.9 mm to (10.9, -135.9)
- moved U20 82.9 mm to (6.41, -140.6)
- moved C54 82.9 mm to (-6.60, -135.4)
- moved J4 82.9 mm to (-9.65, -130.8)
- moved R36 82.9 mm to (9.91, -139.8)
- moved R37 82.9 mm to (3.11, -140.6)
- moved C42 33.1 mm to (135.5, -142.4)
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Connections:
- removed net N$1: D2.ANODE, R12.2
- net TXRX_LED: no longer D2.CATHODE
- net USB_V1: no longer R12.1
Routing:
- net GND: track 176.8 -> 184.7 mm, vias 53 -> 54
- net TXRX_LED: track 8.91 -> 1.28 mm
- net USB_RST: track 24.6 -> 17.5 mm
- net USBDP: track 7.96 -> 2.93 mm
- net USB_V1: track 29.7 -> 25.0 mm
- net FT230_RST: track 26.6 -> 22.0 mm
- net USBDM: track 10.4 -> 6.55 mm
- net N$1: track 1.99 -> 0.00 mm
- net LCD_SDA: track 16.4 -> 15.2 mm
- net LCD_SCL: track 9.56 -> 8.92 mm
Other:
- board outline added: 7.1 x 1.2 mm
