File: Hardware/Octoprober.sch (EAGLE design)
At the start: 180 parts, among them J1 ER-CON2.0-2P-SMD, J4 ER-CON31HT-1, SW1 EVQ-Q2203W, SW2 EVQ-Q2203W, SW3 EVQ-Q2203W, SW4 EVQ-Q2203W, SW5 EVQ-Q2203W, T1 PCC-SMP-V, T2 PCC-SMP-V, T3 PCC-SMP-V, T4 PCC-SMP-V, T5 PCC-SMP-V, T6 PCC-SMP-V, T7 PCC-SMP-V, T8 PCC-SMP-V, U1 P8X32A-Q44, U10 DS1340Z-33+, U11 MAX31856MUD+, U12 MAX31856MUD+, U13 MAX31856MUD+, U14 MAX31856MUD+, U15 MAX31856MUD+, U16 MAX31856MUD+, U17 MAX31856MUD+, U18 MAX31856MUD+, U19 IP4234CZ6,125, U2 CAT24C512WI-GT3, U20 PMV160UP,215, U3 ADP3338AKCZ-3.3-RL, U4 FT230XQ-R, U5 BQ24075RGTT, U6 74HC2G04GV,125, U7 PMV22EN,215, U8 PMV160UP,215, U9 MCP3021A5T-E/OT, X1 ABLS3-6.000MHZ-D4Y-T, X2 ABS25-32.768KHz-1-T

Commit message: starting on the revamp.
Parts:
- removed BATT1: MIKROE-1120, PP_Connectors:PH_1X02HEADER_PTH
- removed FID1: GSM_FIDUCIAL, MF_Aesthetics:GSM_FIDUCIAL
- removed J2: (no value), PP_Connectors:PH_1X04HEADER_PTH
- removed U3: ADP3338AKCZ-3.3-RL, PP_PowerIC:FIXED_VOLTAGE_REGSOT-223_ALT
- added J5: (no value), PP_Connectors:CON_01X02_2.54MM_PIN_HEADER
- added J6: (no value), PP_Connectors:CON_01X02_ER-CON2.0-2P-SMD
- added U21: 74HCT2G04GV,125, PP_DigitalIC:74HCT2G04GV,125
- C1, C35: device PP_Passives:CAPACITOR_NON_POLAR0402 -> PP_Passives:CAPACITOR_NON_POLAR_0402
- C10, C11, C12, C13, C14, C15, C16, C17, C18, C19, C2, C20, C21, C22, C24, C26, C27, C28, C29, C3, C30, C34, C37, C38, C39, C4, C40, C46, C47, C48, C49, C5, C50, C51, C52, C55, C56, C57, C58, C59, C6, C60, C61, C62, C63, C64, C65, C66, C67, C68, C69, C70, C71, C72, C73, C74, C75, C76, C77, C78, C79, C80, C9: device PP_Passives:CAPACITOR_NON_POLAR0603 -> PP_Passives:CAPACITOR_NON_POLAR_0603
- C23, C25, C31, C32, C33, C36, C41, C42, C43, C44, C54, C7, C8: device PP_Passives:CAPACITOR_NON_POLAR1206 -> PP_Passives:CAPACITOR_NON_POLAR_1206
- C45, C53: device PP_Passives:CAPACITOR_POLARIZEDCASE_D -> PP_Passives:CAPACITOR_POLARIZED_CASE_D
- D1, D12, D2: device PP_LED:LED_SINGLE0805 -> PP_LED:LED_SINGLE_0805
- D3: device PP_Passives:DIODESOD-128 -> PP_Passives:DIODE_SOD-128
- J1: value ER-CON2.0-2P-SMD -> (none); device PP_Connectors:PH_1X02ER-CON2.0-2P-SMD -> PP_Connectors:CON_01X04_2.54MM_PIN_HEADER
- J4: device PP_Connectors:ER-CON31HT-1 -> PP_Connectors:CON_01X31_ER-CON31HT-1
- L1, L2, R1, R10, R11, R12, R13, R14, R15, R16, R17, R18, R19, R20, R21, R22, R23, R24, R25, R26, R27, R28, R29, R30, R31, R32, R33, R34, R35, R36, R37, R38, R39, R8, R9: device PP_Passives:RESISTOR0603 -> PP_Passives:RESISTOR_0603
- L18: device PP_Passives:INDUCTORCDRH6D28 -> PP_Passives:INDUCTOR_CDRH6D28
- OP1: device PP_DigitalIC:ACPL-227SOIC-8 -> PP_DigitalIC:ACPL-227-500E
- R2, R3, R4, R5, R6, R7: device PP_Passives:RESISTOR0402 -> PP_Passives:RESISTOR_0402
- SW1, SW2, SW3, SW4, SW5: device PP_Electromechanical:SPSTEVQ-Q2203W -> PP_Electromechanical:SPST_EVQ-Q2203W
- T1, T2, T3, T4, T5, T6, T7, T8: device PP_Connectors:THERMOCOUPLE_CONPCC-SMP-V -> PP_Connectors:THERMOCOUPLE_CON_PCC-SMP-V
- U10: value DS1340Z-33+ -> BQ24075RGTT; device PP_DigitalIC:DS1340SOIC-8 -> PP_PowerIC:BQ2407(5/9)
- U11, U12, U13, U14, U15, U16, U17, U18: device PP_AnalogIC:MAX31856 -> PP_AnalogIC:MAX31856MUD+
- U19: device PP_Passives:IP4234CZ6SOT-457 -> PP_Passives:IP4234CZ6
- U2: device PP_DigitalIC:CAT24M01XI-T2SOIC-8_W -> PP_DigitalIC:EEPROM_I2CSOIC-8
- U20, U8: device PP_DiscreteSemi:MOSFET_P-CHANNEL_SINGLESOT-23 -> PP_DiscreteSemi:MOSFET_P-CHANNEL_SINGLE_SOT-23
- U4: device PP_DigitalIC:FT230XQFN-16 -> PP_DigitalIC:FT230XQ
- U5: value BQ24075RGTT -> ADP3338AKCZ-3.3-RL; device PP_PowerIC:BQ2407XQFN-16 -> PP_PowerIC:LINEAR_VOTLAGE_REGULATORS_ADP3338
- U6: value 74HC2G04GV,125 -> DS1340Z-33+; device PP_DigitalIC:74HCT2G04GV,125TTSOP-6 -> PP_DigitalIC:DS1340Z-33+
- U7: device PP_DiscreteSemi:MOSFET_N-CHANNEL_SINGLESOT-23 -> PP_DiscreteSemi:MOSFET_N-CHANNEL_SINGLE_SOT-23
- U9: device PP_DigitalIC:MCP3021SOT-23A -> PP_DigitalIC:MCP3021A0T-E/OT
- X1: device PP_FreqCtrl:CRYSTALHC-49 -> PP_FreqCtrl:CRYSTAL_HC-49
- X2: device PP_FreqCtrl:CRYSTAL8MM_X_3.8MM -> PP_FreqCtrl:CRYSTAL_8MM_X_3.8MM
Connections:
- net !PWREN: now also U21.2A; no longer U6.2A
- net !SLEEP: now also U21.1A; no longer U6.1A
- net 3.3V: now also U21.VCC, U5.OUT; no longer U10.VCC, U3.OUT
- net A: now also J6.PIN1; no longer J1.1
- net BCD_CHARGER: now also U10.EN2; no longer U5.EN2
- net CHARGING: now also U10.!CHG; no longer U5.!CHG
- net EXT_CON_0: now also J1.1; no longer J2.1
- net EXT_CON_1: now also J1.2; no longer J2.2
- net EXT_CON_2: now also J1.3; no longer J2.3
- net EXT_CON_3: now also J1.4; no longer J2.4
- net GND: now also J5.PIN1, J6.PIN2, U10.SYSOFF, U2.A0, U21.GND, U5.GND, U6.VSS; no longer BATT1.1, J1.2, U3.GND, U5.SYSOFF, U5.VSS, U6.GND
- net ILM: now also U10.ILM; no longer U5.ILM
- net ISET: now also U10.ISET; no longer U5.ISET
- net PGOOD: now also U10.!PGOOD; no longer U5.!PGOOD
- net PWREN: now also U10.EN1, U21.2Y; no longer U5.EN1, U6.2Y
- net RTC_X1: now also U6.X1; no longer U10.X1
- net RTC_X2: now also U6.X2; no longer U10.X2
- net SCL: now also U6.SCL; no longer U10.SCL
- net SDA: now also U6.SDA; no longer U10.SDA
- net SLEEP: now also U10.!CE, U21.1Y; no longer U5.!CE, U6.1Y
- net SYS_V: now also U10.OUT, U6.V_BACK; no longer U10.V_BACK, U5.OUT
- net SYS_V_SW: now also U5.IN; no longer U3.IN
- net TS: now also U10.TS; no longer U5.TS
- net USB_V1: now also U10.IN; no longer U5.IN
- net VBATT: now also J5.PIN2, U10.BAT; no longer BATT1.2, U5.BAT
Other:
- moved on the sheet: C1, C10, C11, C12, C13, C14, C15, C16, C17, C18, C19, C2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

Commit message: Working on new rev. Need to route.
Parts:
- removed J5: (no value), PP_Connectors:CON_01X02_2.54MM_PIN_HEADER
- added BATT1: 1042, PP_Connectors:BATTERY_KEYSTON_1042
- J4: LABEL15 DB6_SCL -> DB6_SDA; LABEL16 DB7_SDA -> DB7_SCL
- J6: value (none) -> ER-CON2.0-2P-SMD
- R10, R11: value 22 -> 27
Connections:
- net GND: now also BATT1.-; no longer J5.PIN1
- net LCD_SCL: now also J4.PIN16, R39.1; no longer J4.PIN11, J4.PIN12, J4.PIN13, J4.PIN15, R38.1
- net LCD_SDA: now also J4.PIN11, J4.PIN12, J4.PIN13, J4.PIN15, R38.1; no longer J4.PIN16, R39.1
- net VBATT: now also BATT1.+; no longer J5.PIN2
Other:
- moved on the sheet: D3

Commit message: Started routing REV3.
Parts:
- removed C41: 10uF, PP_Passives:CAPACITOR_NON_POLAR_1206
- added C81, C82: 47pF, PP_Passives:CAPACITOR_NON_POLAR_0603
- added C83: 0.1uF, PP_Passives:CAPACITOR_NON_POLAR_0603
- X1: value ABLS3-6.000MHZ-D4Y-T -> ABMM-6.000MHZ-B2-T; device PP_FreqCtrl:CRYSTAL_HC-49 -> MF_Frequency_Control:XTL_7MMX5MM
Connections:
- net 3.3V: now also C83.1; no longer C41.1
- net D+: now also C82.1
- net D-: now also C81.1
- net GND: now also C81.2, C82.2, C83.2, X1.GND; no longer C41.2
- net X0: now also X1.X1; no longer X1.P$1
- net X1: now also X1.X0; no longer X1.P$2
Other:
- moved on the sheet: R10, R11

Commit message: More work to check in.
Parts:
- removed D2: 598-8070-107F, PP_LED:LED_SINGLE_0805
- removed R12: 330, PP_Passives:RESISTOR_0603
Connections:
- removed net N$1: D2.ANODE, R12.2
- net TXRX_LED: no longer D2.CATHODE
- net USB_V1: no longer R12.1
Changed lines of the file:
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@@
 <part name="C12" library="PP_Passives" deviceset="CAPACITOR_NON_POLAR" device="_0603" value="0.1uF"/>
 <part name="D1" library="PP_LED" deviceset="LED_SINGLE" device="_0805" value="598-8070-107F"/>
-<part name="D2" library="PP_LED" deviceset="LED_SINGLE" device="_0805" value="598-8070-107F"/>
-<part name="R12" library="PP_Passives" deviceset="RESISTOR" device="_0603" value="330"/>
 <part name="R13" library="PP_Passives" deviceset="RESISTOR" device="_0603" value="330"/>
 <part name="C13" library="PP_Passives" deviceset="CAPACITOR_NON_POLAR" device="_0603" value="0.1uF"/>
@@
 <instance part="C12" gate="G$1" x="-33.02" y="-53.34" rot="R90"/>
 <instance part="D1" gate="G$1" x="-119.38" y="-78.74" rot="R270"/>
-<instance part="D2" gate="G$1" x="-109.22" y="-78.74" rot="R270"/>
-<instance part="R12" gate="G$1" x="-109.22" y="-68.58" rot="R270"/>
 <instance part="R13" gate="G$1" x="-119.38" y="-68.58" rot="R270"/>
 <instance part="C13" gate="G$1" x="-43.18" y="-35.56"/>
@@
 <net name="TXRX_LED" class="0">
 <segment>
-<pinref part="D2" gate="G$1" pin="CATHODE"/>
-<wire x1="-109.22" y1="-81.28" x2="-109.22" y2="-86.36" width="0.1524" layer="91"/>
-<wire x1="-109.22" y1="-86.36" x2="-101.6" y2="-86.36" width="0.1524" layer="91"/>
-<label x="-106.68" y="-86.36" size="0.8128" layer="95" font="vector"/>
-</segment>
-<segment>
 <pinref part="U4" gate="G$1" pin="CBUS0"/>
 <wire x1="-43.18" y1="-60.96" x2="-33.02" y2="-60.96" width="0.1524" layer="91"/>
@@
 <label x="22.86" y="-60.96" size="0.8128" layer="95" font="vector"/>
 <pinref part="U21" gate="G$1" pin="2Y"/>
-</segment>
-</net>
-<net name="N$1" class="0">
-<segment>
-<pinref part="D2" gate="G$1" pin="ANODE"/>
-<pinref part="R12" gate="G$1" pin="2"/>
-<wire x1="-109.22" y1="-76.2" x2="-109.22" y2="-73.66" width="0.1524" layer="91"/>
 </segment>
 </net>
@@
 <pinref part="R13" gate="G$1" pin="1"/>
 <wire x1="-119.38" y1="-63.5" x2="-119.38" y2="-58.42" width="0.1524" layer="91"/>
-<wire x1="-119.38" y1="-58.42" x2="-109.22" y2="-58.42" width="0.1524" layer="91"/>
-<pinref part="R12" gate="G$1" pin="1"/>
-<wire x1="-109.22" y1="-63.5" x2="-109.22" y2="-58.42" width="0.1524" layer="91"/>
-<wire x1="-109.22" y1="-58.42" x2="-101.6" y2="-58.42" width="0.1524" layer="91"/>
+<wire x1="-119.38" y1="-58.42" x2="-101.6" y2="-58.42" width="0.1524" layer="91"/>
 <label x="-106.68" y="-58.42" size="0.8128" layer="95" font="vector"/>
-<junction x="-109.22" y="-58.42"/>
-</segment>
-<segment>
+</segment>
+<segment>
